File: PCB.kicad_pcb (KiCad board)
At the start: 2 copper layers, 7 parts, among them J1 Conn_02x20_Odd_Even, J3 Conn_01x02_Male, J4 Conn_01x02_Male, U1 L298HN, U2 HC-SR04

Commit message: second commit
Connections:
- net GND renamed Net-(J1-Pad30)
- U1 pad 4: +5VD -> Net-(J2-Pad1)
- U1 pad 9: +5VD -> Net-(J2-Pad2)
Changed lines of the file:
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@@
     (zones 0)
     (modules 7)
-    (nets 49)
+    (nets 50)
   )
   (page A4)
@@
   (net 29 "Net-(J1-Pad28)")
   (net 30 "Net-(J1-Pad29)")
-  (net 31 "Net-(J1-Pad31)")
-  (net 32 "Net-(J1-Pad32)")
-  (net 33 "Net-(J1-Pad33)")
-  (net 34 "Net-(J1-Pad34)")
-  (net 35 "Net-(J1-Pad35)")
-  (net 36 "Net-(J1-Pad36)")
-  (net 37 "Net-(J1-Pad37)")
-  (net 38 "Net-(J1-Pad38)")
-  (net 39 "Net-(J1-Pad39)")
-  (net 40 "Net-(J1-Pad40)")
-  (net 41 "Net-(U1-Pad1)")
-  (net 42 "Net-(J3-Pad2)")
-  (net 43 "Net-(J3-Pad1)")
-  (net 44 "Net-(J4-Pad2)")
-  (net 45 "Net-(J4-Pad1)")
-  (net 46 "Net-(U1-Pad15)")
-  (net 47 GND)
-  (net 48 +5VD)
+  (net 31 "Net-(J1-Pad30)")
+  (net 32 "Net-(J1-Pad31)")
+  (net 33 "Net-(J1-Pad32)")
+  (net 34 "Net-(J1-Pad33)")
+  (net 35 "Net-(J1-Pad34)")
+  (net 36 "Net-(J1-Pad35)")
+  (net 37 "Net-(J1-Pad36)")
+  (net 38 "Net-(J1-Pad37)")
+  (net 39 "Net-(J1-Pad38)")
+  (net 40 "Net-(J1-Pad39)")
+  (net 41 "Net-(J1-Pad40)")
+  (net 42 "Net-(U1-Pad1)")
+  (net 43 "Net-(J3-Pad2)")
+  (net 44 "Net-(J3-Pad1)")
+  (net 45 "Net-(J2-Pad1)")
+  (net 46 "Net-(J2-Pad2)")
+  (net 47 "Net-(J4-Pad2)")
+  (net 48 "Net-(J4-Pad1)")
+  (net 49 "Net-(U1-Pad15)")
   (net_class Default "This is the default net class."
     (clearance 0.2)
@@
     (uvia_dia 0.3)
     (uvia_drill 0.1)
-    (add_net +5VD)
-    (add_net GND)
     (add_net "Net-(D1-Pad1)")
     (add_net "Net-(D1-Pad2)")
@@
     (add_net "Net-(J1-Pad29)")
     (add_net "Net-(J1-Pad3)")
+    (add_net "Net-(J1-Pad30)")
     (add_net "Net-(J1-Pad31)")
     (add_net "Net-(J1-Pad32)")
@@
     (add_net "Net-(J1-Pad8)")
     (add_net "Net-(J1-Pad9)")
+    (add_net "Net-(J2-Pad1)")
+    (add_net "Net-(J2-Pad2)")
     (add_net "Net-(J3-Pad1)")
     (add_net "Net-(J3-Pad2)")
@@
       (net 3 "Net-(J1-Pad2)"))
     (pad 4 thru_hole circle (at 3.81 0) (size 1.53 1.53) (drill 1.02) (layers *.Cu *.Mask)
-      (net 39 "Net-(J1-Pad39)"))
+      (net 40 "Net-(J1-Pad39)"))
     (pad 3 thru_hole circle (at 1.27 0) (size 1.53 1.53) (drill 1.02) (layers *.Cu *.Mask)
-      (net 35 "Net-(J1-Pad35)"))
+      (net 36 "Net-(J1-Pad35)"))
     (pad 2 thru_hole circle (at -1.27 0) (size 1.53 1.53) (drill 1.02) (layers *.Cu *.Mask)
-      (net 37 "Net-(J1-Pad37)"))
+      (net 38 "Net-(J1-Pad37)"))
   )
   (module Connector_PinHeader_2.54mm:PinHeader_1x02_P2.54mm_Vertical (layer F.Cu)
@@
     (fp_line (start -0.635 -1.27) (end 1.27 -1.27) (layer F.Fab) (width 0.1))
     (pad 2 thru_hole oval (at 0 2.54) (size 1.7 1.7) (drill 1) (layers *.Cu *.Mask)
-      (net 44 "Net-(J4-Pad2)"))
+      (net 47 "Net-(J4-Pad2)"))
     (pad 1 thru_hole rect (at 0 0) (size 1.7 1.7) (drill 1) (layers *.Cu *.Mask)
-      (net 45 "Net-(J4-Pad1)"))
+      (net 48 "Net-(J4-Pad1)"))
     (model ${KISYS3DMOD}/Connector_PinHeader_2.54mm.3dshapes/PinHeader_1x02_P2.54mm_Vertical.wrl
       (at (xyz 0 0 0))
@@
     (fp_line (start -0.635 -1.27) (end 1.27 -1.27) (layer F.Fab) (width 0.1))
     (pad 2 thru_hole oval (at 0 2.54) (size 1.7 1.7) (drill 1) (layers *.Cu *.Mask)
-      (net 42 "Net-(J3-Pad2)"))
+      (net 43 "Net-(J3-Pad2)"))
     (pad 1 thru_hole rect (at 0 0) (size 1.7 1.7) (drill 1) (layers *.Cu *.Mask)
-      (net 43 "Net-(J3-Pad1)"))
+      (net 44 "Net-(J3-Pad1)"))
     (model ${KISYS3DMOD}/Connector_PinHeader_2.54mm.3dshapes/PinHeader_1x02_P2.54mm_Vertical.wrl
       (at (xyz 0 0 0))
@@
       (net 30 "Net-(J1-Pad29)"))
     (pad 30 thru_hole oval (at 2.54 35.56) (size 1.7 1.7) (drill 1) (layers *.Cu *.Mask)
-      (net 47 GND))
+      (net 31 "Net-(J1-Pad30)"))
     (pad 31 thru_hole oval (at 0 38.1) (size 1.7 1.7) (drill 1) (layers *.Cu *.Mask)
-      (net 31 "Net-(J1-Pad31)"))
+      (net 32 "Net-(J1-Pad31)"))
     (pad 32 thru_hole oval (at 2.54 38.1) (size 1.7 1.7) (drill 1) (layers *.Cu *.Mask)
-      (net 32 "Net-(J1-Pad32)"))
+      (net 33 "Net-(J1-Pad32)"))
     (pad 33 thru_hole oval (at 0 40.64) (size 1.7 1.7) (drill 1) (layers *.Cu *.Mask)
-      (net 33 "Net-(J1-Pad33)"))
+      (net 34 "Net-(J1-Pad33)"))
     (pad 34 thru_hole oval (at 2.54 40.64) (size 1.7 1.7) (drill 1) (layers *.Cu *.Mask)
-      (net 34 "Net-(J1-Pad34)"))
+      (net 35 "Net-(J1-Pad34)"))
     (pad 35 thru_hole oval (at 0 43.18) (size 1.7 1.7) (drill 1) (layers *.Cu *.Mask)
-      (net 35 "Net-(J1-Pad35)"))
+      (net 36 "Net-(J1-Pad35)"))
     (pad 36 thru_hole oval (at 2.54 43.18) (size 1.7 1.7) (drill 1) (layers *.Cu *.Mask)
-      (net 36 "Net-(J1-Pad36)"))
+      (net 37 "Net-(J1-Pad36)"))
     (pad 37 thru_hole oval (at 0 45.72) (size 1.7 1.7) (drill 1) (layers *.Cu *.Mask)
-      (net 37 "Net-(J1-Pad37)"))
+      (net 38 "Net-(J1-Pad37)"))
     (pad 38 thru_hole oval (at 2.54 45.72) (size 1.7 1.7) (drill 1) (layers *.Cu *.Mask)
-      (net 38 "Net-(J1-Pad38)"))
+      (net 39 "Net-(J1-Pad38)"))
     (pad 39 thru_hole oval (at 0 48.26) (size 1.7 1.7) (drill 1) (layers *.Cu *.Mask)
-      (net 39 "Net-(J1-Pad39)"))
+      (net 40 "Net-(J1-Pad39)"))
     (pad 40 thru_hole oval (at 2.54 48.26) (size 1.7 1.7) (drill 1) (layers *.Cu *.Mask)
-      (net 40 "Net-(J1-Pad40)"))
+      (net 41 "Net-(J1-Pad40)"))
     (model ${KISYS3DMOD}/Connector_PinHeader_2.54mm.3dshapes/PinHeader_2x20_P2.54mm_Vertical.wrl
       (at (xyz 0 0 0))
@@
     )
     (pad 1 thru_hole rect (at 0 0) (size 1.8 1.8) (drill 1) (layers *.Cu *.Mask)
-      (net 41 "Net-(U1-Pad1)"))
+      (net 42 "Net-(U1-Pad1)"))
     (pad 2 thru_hole oval (at 1.27 -5.08) (size 1.8 1.8) (drill 1) (layers *.Cu *.Mask)
-      (net 42 "Net-(J3-Pad2)"))
+      (net 43 "Net-(J3-Pad2)"))
     (pad 3 thru_hole oval (at 2.54 0) (size 1.8 1.8) (drill 1) (layers *.Cu *.Mask)
-      (net 43 "Net-(J3-Pad1)"))
+      (net 44 "Net-(J3-Pad1)"))
     (pad 4 thru_hole oval (at 3.81 -5.08) (size 1.8 1.8) (drill 1) (layers *.Cu *.Mask)
-      (net 48 +5VD))
+      (net 45 "Net-(J2-Pad1)"))
     (pad 5 thru_hole oval (at 5.08 0) (size 1.8 1.8) (drill 1) (layers *.Cu *.Mask)
       (net 4 "Net-(J1-Pad3)"))
@@
       (net 6 "Net-(J1-Pad5)"))
     (pad 8 thru_hole oval (at 8.89 -5.08) (size 1.8 1.8) (drill 1) (layers *.Cu *.Mask)
-      (net 47 GND))
+      (net 31 "Net-(J1-Pad30)"))
     (pad 9 thru_hole oval (at 10.16 0) (size 1.8 1.8) (drill 1) (layers *.Cu *.Mask)
-      (net 48 +5VD))
+      (net 46 "Net-(J2-Pad2)"))
     (pad 10 thru_hole oval (at 11.43 -5.08) (size 1.8 1.8) (drill 1) (layers *.Cu *.Mask)
       (net 13 "Net-(J1-Pad12)"))
@@
       (net 17 "Net-(J1-Pad16)"))
     (pad 13 thru_hole oval (at 15.24 0) (size 1.8 1.8) (drill 1) (layers *.Cu *.Mask)
-      (net 44 "Net-(J4-Pad2)"))
+      (net 47 "Net-(J4-Pad2)"))
     (pad 14 thru_hole oval (at 16.51 -5.08) (size 1.8 1.8) (drill 1) (layers *.Cu *.Mask)
-      (net 45 "Net-(J4-Pad1)"))
+      (net 48 "Net-(J4-Pad1)"))
     (pad 15 thru_hole oval (at 17.78 0) (size 1.8 1.8) (drill 1) (layers *.Cu *.Mask)
-      (net 46 "Net-(U1-Pad15)"))
+      (net 49 "Net-(U1-Pad15)"))
     (model ${KISYS3DMOD}/Package_TO_SOT_THT.3dshapes/TO-220-15_P2.54x2.54mm_StaggerOdd_Lead4.58mm_Vertical.wrl
       (at (xyz 0 0 0))
